Commit message: add move_base and other fixes

File: slambot_description/urdf/slambot.urdf.xacro (robot description, xacro)
@@ -21,5 +21,5 @@
     <parent link="base_footprint"/>
     <child link="base_link"/>
-    <origin xyz="0.0 0.0 0.0" rpy="0 0 0"/>
+    <origin xyz="0 0 0" rpy="0 0 0"/>
   </joint>
   <link name="base_link">
